Commit message: Add simulated lidar sensor and warehouse map

File: src/agv_description/urdf/agv.urdf (robot description, URDF)
Before this commit: robot simple_agv, 1 links, 0 joints
Links:
- added link camera_link
- added link laser_link
- link base_link: mass 10 -> None; geometry visual box size=0.6 0.4 0.2
Joints:
- added joint camera_joint: type fixed, parent base_link, child camera_link, origin xyz=0.25 0 0.2 rpy=0 0 0
- added joint laser_joint: type fixed, parent base_link, child laser_link, origin xyz=0.3 0 0.15 rpy=0 0 0
